File: gopro-powerbank.kicad_pcb (KiCad board)
At the start: 2 copper layers, 89.5 x 26.5 mm, 29 parts, among them J1 USB_C_Receptacle_USB2.0, U1 TPS61022RWUR, U2 TP4056, U3 DW01A, U4 8205A, U5 8205A

Commit message: kicad version upgrade
Other:
- net class Default removed
